File: hardware/leds.kicad_sch (KiCad schematic)
At the start: 101 parts

Commit message: Routed half of leds
Parts:
- removed D3: SK6812-EC20, metro-tracker:RGB_LED_2020, symbol metro-tracker:SK6812-EC20
- added C35, C36, C37, C38, C39, C40, C41, C42, C43, C44, C45, C46, C47, C48, C49, C50, C51, C52, C53, C54, C55, C56: 100n, Capacitor_SMD:C_0402_1005Metric, symbol Device:C
- added D5: SK6812-EC20, metro-tracker:RGB_LED_2020, symbol metro-tracker:SK6812-EC20
- renumbered C19 to C16, C20 to C17, C21 to C18, C22 to C19, C23 to C20, C24 to C21, C13 to C22, C14 to C23, C15 to C24, C16 to C25, C17 to C26, C18 to C27, C12 to C28, C11 to C29, C10 to C30, C9 to C31, C8 to C32, C7 to C33, C6 to C34, D8 to D10, D9 to D11, D31 to D12, D32 to D13, D79 to D14, D80 to D15, D81 to D16, D82 to D17, D77 to D18, D78 to D19, D10 to D20, D11 to D21, D12 to D22, D13 to D23, D14 to D24, D15 to D25, D16 to D26, D17 to D27, D18 to D28, D19 to D29, D1 to D3, D20 to D30, D21 to D31, D22 to D32, D23 to D33, D24 to D34, D25 to D35, D26 to D36, D33 to D37, D34 to D38, D35 to D39, D2 to D4, D36 to D40, D37 to D41, D38 to D42, D39 to D43, D40 to D44, D41 to D45, D42 to D46, D43 to D47, D44 to D48, D45 to D49, D46 to D50, D47 to D51, D48 to D52, D49 to D53, D56 to D54, D57 to D55, D58 to D56, D59 to D57, D60 to D58, D61 to D59, D4 to D6, D62 to D60, D63 to D61, D64 to D62, D65 to D63, D66 to D64, D67 to D65, D68 to D66, D69 to D67, D70 to D68, D71 to D69, D5 to D7, D72 to D70, D55 to D71, D30 to D72, D28 to D73, D29 to D74, D74 to D75, D75 to D76, D76 to D77, D51 to D78, D52 to D79, D6 to D8, D53 to D80, D73 to D81, D50 to D82, D27 to D83, D54 to D84, D7 to D9
Connections:
- net +5V: now also C35.1, C36.1, C37.1, C38.1, C39.1, C40.1, C41.1, C42.1, C43.1, C44.1, C45.1, C46.1, C47.1, C48.1, C49.1, C50.1, C51.1, C52.1, C53.1, C54.1, C55.1, C56.1, D5.3 (VDD)
- net DATA_IN: now also D82.2 (DIN); no longer D3.2 (DIN)
- net GND: now also C35.2, C36.2, C37.2, C38.2, C39.2, C40.2, C41.2, C42.2, C43.2, C44.2, C45.2, C46.2, C47.2, C48.2, C49.2, C50.2, C51.2, C52.2, C53.2, C54.2, C55.2, C56.2, D5.1 (VSS)
- net at D71.2 (DIN): now also D49.4 (DOUT); no longer D70.4 (DOUT)
- net at D71.4 (DOUT): now also D79.2 (DIN); no longer D72.2 (DIN)
- net at D76.2 (DIN): no longer D75.4 (DOUT)
- net at D76.4 (DOUT): no longer D77.2 (DIN)
- net at D28.2 (DIN): no longer D27.4 (DOUT)
- net at D28.4 (DOUT): no longer D29.2 (DIN)
- net at D46.2 (DIN): now also D12.4 (DOUT); no longer D45.4 (DOUT)
- net at D46.4 (DOUT): now also D41.2 (DIN); no longer D47.2 (DIN)
- net at D72.4 (DOUT): now also D35.2 (DIN); no longer D73.2 (DIN)
- net at D53.2 (DIN): no longer D52.4 (DOUT)
- net at D53.4 (DOUT): no longer D54.2 (DIN)
- net at D18.2 (DIN): no longer D17.4 (DOUT)
- net at D18.4 (DOUT): no longer D19.2 (DIN)
- net at D78.4 (DOUT): no longer D79.2 (DIN)
- net at D79.4 (DOUT): now also D57.2 (DIN); no longer D80.2 (DIN)
- net at D8.4 (DOUT): now also D11.2 (DIN); no longer D9.2 (DIN)
- net at D50.2 (DIN): now also D82.4 (DOUT); no longer D49.4 (DOUT)
- net at D50.4 (DOUT): now also D9.2 (DIN); no longer D51.2 (DIN)
- net at D38.2 (DIN): now also D74.4 (DOUT); no longer D37.4 (DOUT)
- net at D48.2 (DIN): no longer D47.4 (DOUT)
- net at D48.4 (DOUT): no longer D49.2 (DIN)
- net at D15.2 (DIN): no longer D14.4 (DOUT)
- net at D15.4 (DOUT): no longer D16.2 (DIN)
- net at D80.4 (DOUT): no longer D81.2 (DIN)
- net at D17.2 (DIN): no longer D16.4 (DOUT)
- net at D77.4 (DOUT): no longer D78.2 (DIN)
- net at D33.4 (DOUT): now also D72.2 (DIN); no longer D34.2 (DIN)
- net at D34.4 (DOUT): now also D33.2 (DIN); no longer D35.2 (DIN)
- net at D29.4 (DOUT): now also D27.2 (DIN); no longer D30.2 (DIN)
- net at D52.2 (DIN): now also D41.4 (DOUT); no longer D51.4 (DOUT)
- net at D40.4 (DOUT): now also D12.2 (DIN); no longer D41.2 (DIN)
- net at D42.2 (DIN): now also D39.4 (DOUT); no longer D41.4 (DOUT)
- net at D14.2 (DIN): no longer D13.4 (DOUT)
- net at D30.4 (DOUT): no longer D31.2 (DIN)
- net at D68.2 (DIN): now also D63.4 (DOUT); no longer D67.4 (DOUT)
- net at D68.4 (DOUT): now also D67.2 (DIN); no longer D69.2 (DIN)
- net at D32.4 (DOUT): now also D73.2 (DIN); no longer D33.2 (DIN)
- net at D40.2 (DIN): now also D35.4 (DOUT); no longer D39.4 (DOUT)
- net at D56.4 (DOUT): no longer D57.2 (DIN)
- net at D57.4 (DOUT): now also D54.2 (DIN); no longer D58.2 (DIN)
- net at D43.4 (DOUT): now also D5.2 (DIN); no longer D44.2 (DIN)
- net at D44.4 (DOUT): no longer D45.2 (DIN)
- net at D21.4 (DOUT): now also D25.2 (DIN); no longer D22.2 (DIN)
- net at D83.2 (DIN): no longer D82.4 (DOUT)
- net at D83.4 (DOUT): no longer D84.2 (DIN)
- net at D64.2 (DIN): now also D59.4 (DOUT); no longer D63.4 (DOUT)
- net at D64.4 (DOUT): now also D63.2 (DIN); no longer D65.2 (DIN)
- net at D20.2 (DIN): now also D10.4 (DOUT); no longer D19.4 (DOUT)
- net at D59.2 (DIN): now also D61.4 (DOUT); no longer D58.4 (DOUT)
- net at D60.2 (DIN): no longer D59.4 (DOUT)
- net at D62.4 (DOUT): no longer D63.2 (DIN)
- net at D75.2 (DIN): now also D67.4 (DOUT); no longer D74.4 (DOUT)
- net at D26.4 (DOUT): now also D31.2 (DIN); no longer D27.2 (DIN)
- net at D55.4 (DOUT): now also D58.2 (DIN); no longer D56.2 (DIN)
- net at D61.2 (DIN): now also D58.4 (DOUT); no longer D60.4 (DOUT)
- net at D62.2 (DIN): no longer D61.4 (DOUT)
- net at D11.4 (DOUT): now also D22.2 (DIN); no longer D12.2 (DIN)
- net at D36.2 (DIN): no longer D35.4 (DOUT)
- net at D36.4 (DOUT): no longer D37.2 (DIN)
- net at D7.2 (DIN): now also D4.4 (DOUT); no longer D6.4 (DOUT)
- net at D6.2 (DIN): now also D5.4 (DOUT)
- net at D66.2 (DIN): no longer D65.4 (DOUT)
- net at D66.4 (DOUT): no longer D67.2 (DIN)
- net at D81.4 (DOUT): now also D19.2 (DIN); no longer D82.2 (DIN)
- net at D13.2 (DIN): no longer D12.4 (DOUT)
- net at D69.4 (DOUT): no longer D70.2 (DIN)
- net at D24.4 (DOUT): now also D29.2 (DIN); no longer D25.2 (DIN)
- new net: D27.4 (DOUT), D34.2 (DIN)
- new net: D49.2 (DIN), D52.4 (DOUT)
- new net: D75.4 (DOUT), D81.2 (DIN)
- new net: D16.2 (DIN), D19.4 (DOUT)
- new net: D3.2 (DIN), D6.4 (DOUT)
Other:
- moved on the sheet: C16, C17, C18, C19, C20, C21, C22, C23, C24, C25, C26, C27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
