File: hardware/leds.kicad_sch (KiCad schematic)
At the start: 123 parts

Commit message: Updated LED footprint
Connections:
- net +5V: now also D10.1 (VDD), D11.1 (VDD), D12.1 (VDD), D13.1 (VDD), D14.1 (VDD), D15.1 (VDD), D16.1 (VDD), D17.1 (VDD), D18.1 (VDD), D19.1 (VDD), D20.1 (VDD), D21.1 (VDD), D22.1 (VDD), D23.1 (VDD), D24.1 (VDD), D25.1 (VDD), D26.1 (VDD), D27.1 (VDD), D28.1 (VDD), D29.1 (VDD), D3.1 (VDD), D30.1 (VDD), D31.1 (VDD), D32.1 (VDD), D33.1 (VDD), D34.1 (VDD), D35.1 (VDD), D36.1 (VDD), D37.1 (VDD), D38.1 (VDD), D39.1 (VDD), D4.1 (VDD), D40.1 (VDD), D41.1 (VDD), D42.1 (VDD), D43.1 (VDD), D44.1 (VDD), D45.1 (VDD), D46.1 (VDD), D47.1 (VDD), D48.1 (VDD), D49.1 (VDD), D5.1 (VDD), D50.1 (VDD), D51.1 (VDD), D52.1 (VDD), D53.1 (VDD), D54.1 (VDD), D55.1 (VDD), D56.1 (VDD), D57.1 (VDD), D58.1 (VDD), D59.1 (VDD), D6.1 (VDD), D60.1 (VDD), D61.1 (VDD), D62.1 (VDD), D63.1 (VDD), D64.1 (VDD), D65.1 (VDD), D66.1 (VDD), D67.1 (VDD), D68.1 (VDD), D69.1 (VDD), D7.1 (VDD), D70.1 (VDD), D71.1 (VDD), D72.1 (VDD), D73.1 (VDD), D74.1 (VDD), D75.1 (VDD), D76.1 (VDD), D77.1 (VDD), D78.1 (VDD), D79.1 (VDD), D8.1 (VDD), D80.1 (VDD), D81.1 (VDD), D82.1 (VDD), D83.1 (VDD), D84.1 (VDD), D9.1 (VDD); no longer D10.3 (VDD), D11.3 (VDD), D12.3 (VDD), D13.3 (VDD), D14.3 (VDD), D15.3 (VDD), D16.3 (VDD), D17.3 (VDD), D18.3 (VDD), D19.3 (VDD), D20.3 (VDD), D21.3 (VDD), D22.3 (VDD), D23.3 (VDD), D24.3 (VDD), D25.3 (VDD), D26.3 (VDD), D27.3 (VDD), D28.3 (VDD), D29.3 (VDD), D3.3 (VDD), D30.3 (VDD), D31.3 (VDD), D32.3 (VDD), D33.3 (VDD), D34.3 (VDD), D35.3 (VDD), D36.3 (VDD), D37.3 (VDD), D38.3 (VDD), D39.3 (VDD), D4.3 (VDD), D40.3 (VDD), D41.3 (VDD), D42.3 (VDD), D43.3 (VDD), D44.3 (VDD), D45.3 (VDD), D46.3 (VDD), D47.3 (VDD), D48.3 (VDD), D49.3 (VDD), D5.3 (VDD), D50.3 (VDD), D51.3 (VDD), D52.3 (VDD), D53.3 (VDD), D54.3 (VDD), D55.3 (VDD), D56.3 (VDD), D57.3 (VDD), D58.3 (VDD), D59.3 (VDD), D6.3 (VDD), D60.3 (VDD), D61.3 (VDD), D62.3 (VDD), D63.3 (VDD), D64.3 (VDD), D65.3 (VDD), D66.3 (VDD), D67.3 (VDD), D68.3 (VDD), D69.3 (VDD), D7.3 (VDD), D70.3 (VDD), D71.3 (VDD), D72.3 (VDD), D73.3 (VDD), D74.3 (VDD), D75.3 (VDD), D76.3 (VDD), D77.3 (VDD), D78.3 (VDD), D79.3 (VDD), D8.3 (VDD), D80.3 (VDD), D81.3 (VDD), D82.3 (VDD), D83.3 (VDD), D84.3 (VDD), D9.3 (VDD)
- net DATA_IN: now also D82.4 (DIN); no longer D82.2 (DIN)
- net GND: now also D10.3 (VSS), D11.3 (VSS), D12.3 (VSS), D13.3 (VSS), D14.3 (VSS), D15.3 (VSS), D16.3 (VSS), D17.3 (VSS), D18.3 (VSS), D19.3 (VSS), D20.3 (VSS), D21.3 (VSS), D22.3 (VSS), D23.3 (VSS), D24.3 (VSS), D25.3 (VSS), D26.3 (VSS), D27.3 (VSS), D28.3 (VSS), D29.3 (VSS), D3.3 (VSS), D30.3 (VSS), D31.3 (VSS), D32.3 (VSS), D33.3 (VSS), D34.3 (VSS), D35.3 (VSS), D36.3 (VSS), D37.3 (VSS), D38.3 (VSS), D39.3 (VSS), D4.3 (VSS), D40.3 (VSS), D41.3 (VSS), D42.3 (VSS), D43.3 (VSS), D44.3 (VSS), D45.3 (VSS), D46.3 (VSS), D47.3 (VSS), D48.3 (VSS), D49.3 (VSS), D5.3 (VSS), D50.3 (VSS), D51.3 (VSS), D52.3 (VSS), D53.3 (VSS), D54.3 (VSS), D55.3 (VSS), D56.3 (VSS), D57.3 (VSS), D58.3 (VSS), D59.3 (VSS), D6.3 (VSS), D60.3 (VSS), D61.3 (VSS), D62.3 (VSS), D63.3 (VSS), D64.3 (VSS), D65.3 (VSS), D66.3 (VSS), D67.3 (VSS), D68.3 (VSS), D69.3 (VSS), D7.3 (VSS), D70.3 (VSS), D71.3 (VSS), D72.3 (VSS), D73.3 (VSS), D74.3 (VSS), D75.3 (VSS), D76.3 (VSS), D77.3 (VSS), D78.3 (VSS), D79.3 (VSS), D8.3 (VSS), D80.3 (VSS), D81.3 (VSS), D82.3 (VSS), D83.3 (VSS), D84.3 (VSS), D9.3 (VSS); no longer D10.1 (VSS), D11.1 (VSS), D12.1 (VSS), D13.1 (VSS), D14.1 (VSS), D15.1 (VSS), D16.1 (VSS), D17.1 (VSS), D18.1 (VSS), D19.1 (VSS), D20.1 (VSS), D21.1 (VSS), D22.1 (VSS), D23.1 (VSS), D24.1 (VSS), D25.1 (VSS), D26.1 (VSS), D27.1 (VSS), D28.1 (VSS), D29.1 (VSS), D3.1 (VSS), D30.1 (VSS), D31.1 (VSS), D32.1 (VSS), D33.1 (VSS), D34.1 (VSS), D35.1 (VSS), D36.1 (VSS), D37.1 (VSS), D38.1 (VSS), D39.1 (VSS), D4.1 (VSS), D40.1 (VSS), D41.1 (VSS), D42.1 (VSS), D43.1 (VSS), D44.1 (VSS), D45.1 (VSS), D46.1 (VSS), D47.1 (VSS), D48.1 (VSS), D49.1 (VSS), D5.1 (VSS), D50.1 (VSS), D51.1 (VSS), D52.1 (VSS), D53.1 (VSS), D54.1 (VSS), D55.1 (VSS), D56.1 (VSS), D57.1 (VSS), D58.1 (VSS), D59.1 (VSS), D6.1 (VSS), D60.1 (VSS), D61.1 (VSS), D62.1 (VSS), D63.1 (VSS), D64.1 (VSS), D65.1 (VSS), D66.1 (VSS), D67.1 (VSS), D68.1 (VSS), D69.1 (VSS), D7.1 (VSS), D70.1 (VSS), D71.1 (VSS), D72.1 (VSS), D73.1 (VSS), D74.1 (VSS), D75.1 (VSS), D76.1 (VSS), D77.1 (VSS), D78.1 (VSS), D79.1 (VSS), D8.1 (VSS), D80.1 (VSS), D81.1 (VSS), D82.1 (VSS), D83.1 (VSS), D84.1 (VSS), D9.1 (VSS)
- net at D71.2 (DOUT): now also D79.4 (DIN); no longer D49.4 (DOUT)
- net at D71.4 (DIN): now also D49.2 (DOUT); no longer D79.2 (DIN)
- net at D46.2 (DOUT): now also D41.4 (DIN); no longer D12.4 (DOUT)
- net at D46.4 (DIN): now also D12.2 (DOUT); no longer D41.2 (DIN)
- net at D72.2 (DOUT): now also D35.4 (DIN); no longer D33.4 (DOUT)
- net at D72.4 (DIN): now also D33.2 (DOUT); no longer D35.2 (DIN)
- net at D57.2 (DOUT): now also D54.4 (DIN); no longer D79.4 (DOUT)
- net at D8.2 (DOUT): now also D11.4 (DIN); no longer D7.4 (DOUT)
- net at D8.4 (DIN): now also D7.2 (DOUT); no longer D11.2 (DIN)
- net at D50.2 (DOUT): now also D9.4 (DIN); no longer D82.4 (DOUT)
- net at D50.4 (DIN): now also D82.2 (DOUT); no longer D9.2 (DIN)
- net at D38.2 (DOUT): now also D39.4 (DIN); no longer D74.4 (DOUT)
- net at D38.4 (DIN): now also D74.2 (DOUT); no longer D39.2 (DIN)
- net at D73.2 (DOUT): now also D74.4 (DIN); no longer D32.4 (DOUT)
- net at D73.4 (DIN): now also D32.2 (DOUT); no longer D74.2 (DIN)
- net at D34.2 (DOUT): now also D33.4 (DIN); no longer D27.4 (DOUT)
- net at D34.4 (DIN): now also D27.2 (DOUT); no longer D33.2 (DIN)
- net at D29.2 (DOUT): now also D27.4 (DIN); no longer D24.4 (DOUT)
- net at D29.4 (DIN): now also D24.2 (DOUT); no longer D27.2 (DIN)
- net at D52.2 (DOUT): now also D49.4 (DIN); no longer D41.4 (DOUT)
- net at D52.4 (DIN): now also D41.2 (DOUT); no longer D49.2 (DIN)
- net at D23.2 (DOUT): now also D24.4 (DIN); no longer D22.4 (DOUT)
- net at D23.4 (DIN): now also D22.2 (DOUT); no longer D24.2 (DIN)
- net at D68.2 (DOUT): now also D67.4 (DIN); no longer D63.4 (DOUT)
- net at D68.4 (DIN): now also D63.2 (DOUT); no longer D67.2 (DIN)
- net at D31.4 (DIN): now also D26.2 (DOUT); no longer D32.2 (DIN)
- net at D42.2 (DOUT): now also D43.4 (DIN); no longer D39.4 (DOUT)
- net at D5.2 (DOUT): now also D6.4 (DIN); no longer D43.4 (DOUT)
- net at D5.4 (DIN): now also D43.2 (DOUT); no longer D6.2 (DIN)
- net at D57.4 (DIN): now also D79.2 (DOUT); no longer D54.2 (DIN)
- net at D42.4 (DIN): now also D39.2 (DOUT); no longer D43.2 (DIN)
- net at D21.2 (DOUT): now also D25.4 (DIN); no longer D20.4 (DOUT)
- net at D21.4 (DIN): now also D20.2 (DOUT); no longer D25.2 (DIN)
- net at D64.2 (DOUT): now also D63.4 (DIN); no longer D59.4 (DOUT)
- net at D64.4 (DIN): now also D59.2 (DOUT); no longer D63.2 (DIN)
- net at D10.4 (DIN): now also D9.2 (DOUT); no longer D20.2 (DIN)
- net at D10.2 (DOUT): now also D20.4 (DIN); no longer D9.4 (DOUT)
- net at D61.4 (DIN): now also D58.2 (DOUT); no longer D59.2 (DIN)
- net at D75.2 (DOUT): now also D81.4 (DIN); no longer D67.4 (DOUT)
- net at D75.4 (DIN): now also D67.2 (DOUT); no longer D81.2 (DIN)
- net at D31.2 (DOUT): now also D32.4 (DIN); no longer D26.4 (DOUT)
- net at D16.2 (DOUT): no longer D19.4 (DOUT)
- net at D16.4 (DIN): now also D19.2 (DOUT)
- net at D55.2 (DOUT): now also D58.4 (DIN); no longer D54.4 (DOUT)
- net at D55.4 (DIN): now also D54.2 (DOUT); no longer D58.2 (DIN)
- net at D61.2 (DOUT): now also D59.4 (DIN); no longer D58.4 (DOUT)
- net at D4.4 (DIN): now also D3.2 (DOUT); no longer D7.2 (DIN)
- net at D4.2 (DOUT): now also D7.4 (DIN); no longer D3.4 (DOUT)
- net at D40.4 (DIN): now also D35.2 (DOUT); no longer D12.2 (DIN)
- net at D40.2 (DOUT): now also D12.4 (DIN); no longer D35.4 (DOUT)
- new net: D25.2 (DOUT), D26.4 (DIN)
- new net: D11.2 (DOUT), D22.4 (DIN)
- new net: D3.4 (DIN), D6.2 (DOUT)
- new net: D19.4 (DIN), D81.2 (DOUT)

Commit message: Initial routing done
Connections:
- net at D76.2 (DOUT): now also D70.4 (DIN)
- net at D76.4 (DIN): now also D77.2 (DOUT)
- net at D28.2 (DOUT): now also D30.4 (DIN)
- net at D28.4 (DIN): now also D47.2 (DOUT)
- net at D53.2 (DOUT): now also D51.4 (DIN)
- net at D53.4 (DIN): now also D78.2 (DOUT)
- net at D18.2 (DOUT): now also D77.4 (DIN)
- net at D18.4 (DIN): now also D14.2 (DOUT)
- net at D48.2 (DOUT): now also D47.4 (DIN)
- net at D48.4 (DIN): now also D51.2 (DOUT)
- net at D15.2 (DOUT): now also D17.4 (DIN)
- net at D15.4 (DIN): now also D16.2 (DOUT)
- net at D80.2 (DOUT): now also D56.4 (DIN)
- net at D80.4 (DIN): now also D60.2 (DOUT)
- net at D17.2 (DOUT): now also D14.4 (DIN)
- net at D30.2 (DOUT): now also D36.4 (DIN)
- net at D44.2 (DOUT): now also D45.4 (DIN)
- net at D44.4 (DIN): now also D37.2 (DOUT)
- net at D83.2 (DOUT): now also D13.4 (DIN)
- net at D83.4 (DIN): now also D36.2 (DOUT)
- net at D62.2 (DOUT): now also D60.4 (DIN)
- net at D62.4 (DIN): now also D65.2 (DOUT)
- net at D66.2 (DOUT): now also D65.4 (DIN)
- net at D66.4 (DIN): now also D69.2 (DOUT)
- net at D56.2 (DOUT): now also D84.4 (DIN)
- net at D13.2 (DOUT): now also D37.4 (DIN)
- net at D69.4 (DIN): now also D70.2 (DOUT)
- net at D84.2 (DOUT): now also D78.4 (DIN)
Other:
- moved on the sheet: D13, D14, D15, D17, D18, D28, D30, D36, D37, D44, D45, D47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

Commit message: added buttons
Other:
- moved on the sheet: C16, C17, C18, C19, C20, C21, C22, C23, C24, C25, C26, C27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
