File: hardware/metromap.kicad_sch (KiCad schematic)
At the start: 36 parts, among them J1 USB_C_Receptacle_USB2.0_16P, U1 AZ1117-3.3, U2 ESP32-C6-MINI-1-H4, U3 SN74LVC1G125DBV

Commit message: Routed half of leds
Parts:
- renumbered C34 to C1, C26 to C10, C28 to C11, C29 to C12, C30 to C13, C31 to C14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
