File: hardware/metromap.kicad_sch (KiCad schematic)
At the start: 55 parts, among them J1 USB_C_Receptacle_USB2.0_16P, SW1 XUNPU_TS-1088-AR02016, SW2 XUNPU_TS-1088-AR02016, U1 AZ1117-3.3, U2 SN74AHCT1G125DBVR, U3 ESP32-C6-MINI-1-H4, U4 CH221K, U5 VEML7700-TR, U6 AP2112K-3.3, U7 SRV05-4

Commit message: Fill in missing JLCPCB part numbers
- Add JLCPCB part number and MPN fields for R1, R2, R6, R8-R16, C57,
  C60, SW1, SW2, U2, U4, U5 and U6 (schematic and PCB)
- Correct C8/C59 value to 100u to match C3339
- Exclude test points TP1-TP4 from BOM and position files

Co-Authored-By: Claude Opus 5.5 <noreply@anthropic.com>
Claude-Session: https://claude.ai/code/session_014z6apRKr3hCTmHGSZGi3ao
Parts:
- C57, C60: JLCPCB Part Number (none) -> C15849; Manufacturer Part Name JLCPCB (none) -> CL10A105KB8NNNC
- C59, C8: value 47u -> 100u
- R1, R10, R13, R14, R15, R16, R2: JLCPCB Part Number (none) -> C25804; Manufacturer Part Name JLCPCB (none) -> 0603WAF1002T5E
- R11, R12: JLCPCB Part Number (none) -> C23162; Manufacturer Part Name JLCPCB (none) -> 0603WAF4701T5E
- R6: JLCPCB Part Number (none) -> C23140; Manufacturer Part Name JLCPCB (none) -> 0603WAF330JT5E
- R8: JLCPCB Part Number (none) -> C25803; Manufacturer Part Name JLCPCB (none) -> 0603WAF1003T5E
- R9: JLCPCB Part Number (none) -> C21190; Manufacturer Part Name JLCPCB (none) -> 0603WAF1001T5E
- SW1, SW2: JLCPCB Part Number (none) -> C720477; Manufacturer Part Name JLCPCB (none) -> TS-1088-AR02016
- TP1, TP2, TP3, TP4: now left out of the parts list
- U2: JLCPCB Part Number (none) -> C7484; Manufacturer Part Name JLCPCB (none) -> SN74AHCT1G125DBVR
- U4: JLCPCB Part Number (none) -> C5125736; Manufacturer Part Name JLCPCB (none) -> CH221K
- U5: JLCPCB Part Number (none) -> C504893; Manufacturer Part Name JLCPCB (none) -> VEML7700-TR
- U6: JLCPCB Part Number (none) -> C51118; Manufacturer Part Name JLCPCB (none) -> AP2112K-3.3TRG1
