File: hardware/metromap.kicad_pcb (KiCad board)
At the start: 4 copper layers, 100 x 100 mm, 179 parts, among them J1 USB_C_Receptacle_USB2.0_16P, SW1 XUNPU_TS-1088-AR02016, SW2 XUNPU_TS-1088-AR02016, U1 AZ1117-3.3, U2 SN74AHCT1G125DBVR, U3 ESP32-C6-MINI-1-H4, U4 CH221K, U5 VEML7700-TR, U6 AP2112K-3.3, U7 SRV05-4

Commit message: fix polyfuse
Parts:
- F1: value Polyfuse -> 3A
- moved C60 0.30 mm to (82.2, 108.5)
- moved R1 0.30 mm to (82.2, 105.5)
- moved SW1 0.23 mm to (79.4, 109.0)
- turned SW2 to 180 degrees
Connections:
- SW2 pad 1: Net-(U3-IO9) -> GND
- SW2 pad 2: GND -> Net-(U3-IO9)
Routing:
- net /CON_USB_D-: track 7.98 -> 10.3 mm
- net /CON_USB_D+: track 8.91 -> 11.2 mm
- net /EN: track 9.02 -> 8.46 mm
- net GND: vias 165 -> 164
