File: hardware/metromap.kicad_pcb (KiCad board)
At the start: 4 copper layers, 100 x 100 mm, 179 parts, among them J1 USB_C_Receptacle_USB2.0_16P, SW1 XUNPU_TS-1088-AR02016, SW2 XUNPU_TS-1088-AR02016, U1 AZ1117-3.3, U2 SN74AHCT1G125DBVR, U3 ESP32-C6-MINI-1-H4, U4 CH221K, U5 VEML7700-TR, U6 AP2112K-3.3, U7 SRV05-4

Commit message: Fill in missing JLCPCB part numbers
- Add JLCPCB part number and MPN fields for R1, R2, R6, R8-R16, C57,
  C60, SW1, SW2, U2, U4, U5 and U6 (schematic and PCB)
- Correct C8/C59 value to 100u to match C3339
- Exclude test points TP1-TP4 from BOM and position files

Co-Authored-By: Claude Opus 5.5 <noreply@anthropic.com>
Claude-Session: https://claude.ai/code/session_014z6apRKr3hCTmHGSZGi3ao
Parts:
- C59, C8: value 47u -> 100u
